File: schematics/tmc-260-shield.brd (EAGLE design)
At the start: 68.6 x 53.3 mm, 64 parts, among them IC1 TMC260-PA, J1 POWER_JACKPTH, Q1 BC856SOT323, T2 BC850SOT323, T3 BC850SOT323, T4 BC850SOT323

Commit message: adding capacitor values
Parts:
- C1, C2: value (none) -> Elko Panasonic G, 50V, EEEFC1H470P / EEEFK1H221P
- C1': value (none) -> TTH alternative to C1
- C2': value (none) -> TTH alternative to C2
- C3, C4, C5, C6, C8: value (none) -> 1µF,50V
Changed lines of the file:
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@@
 <?xml version="1.0" encoding="utf-8"?>
 <!DOCTYPE eagle SYSTEM "eagle.dtd">
-<eagle version="6.4">
+<eagle version="6.3">
 <drawing>
 <settings>
@@
 <attribute name="VALUE" x="-0.675" y="25.4" size="1.016" layer="27" rot="R180"/>
 </element>
-<element name="C2" library="rc-master" package="CSV-G" value="" x="24.98" y="18.985" smashed="yes" rot="R90">
+<element name="C2" library="rc-master" package="CSV-G" value="Elko Panasonic G, 50V, EEEFC1H470P / EEEFK1H221P" x="24.98" y="18.985" smashed="yes" rot="R90">
 <attribute name="NAME" x="23.7" y="25.54" size="0.8128" layer="25" ratio="18" rot="R180"/>
 <attribute name="VALUE" x="28.4725" y="24.7" size="0.8128" layer="27" ratio="10" rot="R90"/>
 </element>
-<element name="C1" library="rc-master" package="CSV-G" value="" x="13.925" y="18.985" smashed="yes" rot="R90">
+<element name="C1" library="rc-master" package="CSV-G" value="Elko Panasonic G, 50V, EEEFC1H470P / EEEFK1H221P" x="13.925" y="18.985" smashed="yes" rot="R90">
 <attribute name="NAME" x="17.1" y="25.485" size="0.8128" layer="25" ratio="18" rot="R180"/>
 <attribute name="VALUE" x="17.4175" y="24.7" size="0.8128" layer="27" ratio="10" rot="R90"/>
@@
 </element>
 <element name="R9" library="rc-master-smd" package="R0603" value="10k" x="8" y="33.5" rot="R270"/>
-<element name="C8" library="rc-master-smd" package="C0603" value="" x="6.6" y="22.445" smashed="yes" rot="R180">
+<element name="C8" library="rc-master-smd" package="C0603" value="1µF,50V" x="6.6" y="22.445" smashed="yes" rot="R180">
 <attribute name="NAME" x="3.451" y="21.746" size="0.8128" layer="25" ratio="18"/>
 <attribute name="VALUE" x="8.124" y="23.969" size="0.6096" layer="27" ratio="10" rot="R180"/>
@@
 <element name="R17" library="rc-master-smd" package="R0603" value="100k" x="11" y="44" rot="R270"/>
 <element name="U$10" library="molex-kk" package="KK-H-4" value="KK4H" x="56.5" y="23.5" smashed="yes"/>
-<element name="C3" library="rc-master-smd" package="C0603" value="" x="49.2" y="34.975" smashed="yes" rot="R180">
+<element name="C3" library="rc-master-smd" package="C0603" value="1µF,50V" x="49.2" y="34.975" smashed="yes" rot="R180">
 <attribute name="NAME" x="49.826" y="33.291" size="0.8128" layer="25" ratio="18"/>
 <attribute name="VALUE" x="50.724" y="36.499" size="0.6096" layer="27" ratio="10" rot="R180"/>
@@
 <attribute name="NAME" x="47.392" y="2.87" size="0.8128" layer="25" ratio="18"/>
 </element>
-<element name="C4" library="rc-master-smd" package="C0603" value="" x="52" y="24.25" smashed="yes" rot="R180">
+<element name="C4" library="rc-master-smd" package="C0603" value="1µF,50V" x="52" y="24.25" smashed="yes" rot="R180">
 <attribute name="NAME" x="48.976" y="23.766" size="0.8128" layer="25" ratio="18"/>
 <attribute name="VALUE" x="53.524" y="25.774" size="0.6096" layer="27" ratio="10" rot="R180"/>
 </element>
-<element name="C5" library="rc-master-smd" package="C0603" value="" x="53" y="27" smashed="yes" rot="R90">
+<element name="C5" library="rc-master-smd" package="C0603" value="1µF,50V" x="53" y="27" smashed="yes" rot="R90">
 <attribute name="NAME" x="51.316" y="30.124" size="0.8128" layer="25" ratio="18" rot="R270"/>
 <attribute name="VALUE" x="54.524" y="25.476" size="0.6096" layer="27" ratio="10" rot="R90"/>
 </element>
-<element name="C6" library="rc-master-smd" package="C1206" value="" x="50.9" y="21.9" rot="R180"/>
+<element name="C6" library="rc-master-smd" package="C1206" value="1µF,50V" x="50.9" y="21.9" rot="R180"/>
 <element name="VMOT" library="SparkFun" package="1X02_NO_SILK" value="" x="1.89" y="18.14" smashed="yes">
 <attribute name="NAME" x="0.9438" y="19.3688" size="1.016" layer="25"/>
 <attribute name="VALUE" x="0.62" y="14.965" size="1.27" layer="27"/>
 </element>
-<element name="C2'" library="rc-master" package="CE-035X100" value="" x="13.95" y="19" smashed="yes">
+<element name="C2'" library="rc-master" package="CE-035X100" value="TTH alternative to C2" x="13.95" y="19" smashed="yes">
 <attribute name="VALUE" x="11.0925" y="15.5075" size="0.8128" layer="27" ratio="10"/>
 </element>
-<element name="C1'" library="rc-master" package="CE-035X100" value="" x="25" y="19" smashed="yes">
+<element name="C1'" library="rc-master" package="CE-035X100" value="TTH alternative to C1" x="25" y="19" smashed="yes">
 <attribute name="VALUE" x="22.1425" y="15.5075" size="0.8128" layer="27" ratio="10"/>
 </element>

Commit message: Fixed some capacitor values
C6: changed value from 1µF to 10µF
C7: added value 1µF
C9: added value 1µF
C10: changed from 10µF to 1µF
Parts:
- C10: value 10µF -> 1µF
- C6: value 1µF,50V -> 10µF,50V
- C7, C9: value (none) -> 1µF
Changed lines of the file:
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@@
 <attribute name="VALUE" x="38.789" y="12.941" size="0.6096" layer="27" ratio="10" rot="R90"/>
 </element>
-<element name="C7" library="rc-master-smd" package="C0603" value="" x="51.24" y="27.005" smashed="yes" rot="R90">
+<element name="C7" library="rc-master-smd" package="C0603" value="1µF" x="51.24" y="27.005" smashed="yes" rot="R90">
 <attribute name="NAME" x="50.376" y="30.119" size="0.8128" layer="25" ratio="18" rot="R270"/>
 <attribute name="VALUE" x="52.764" y="25.481" size="0.6096" layer="27" ratio="10" rot="R90"/>
 </element>
-<element name="C9" library="rc-master-smd" package="C0603" value="" x="52.98" y="30.44" smashed="yes" rot="R90">
+<element name="C9" library="rc-master-smd" package="C0603" value="1µF" x="52.98" y="30.44" smashed="yes" rot="R90">
 <attribute name="NAME" x="53.784" y="32.864" size="0.8128" layer="25" ratio="18" rot="R180"/>
 <attribute name="VALUE" x="54.504" y="28.916" size="0.6096" layer="27" ratio="10" rot="R90"/>
 </element>
-<element name="C10" library="rc-master-smd" package="C0603" value="10µF" x="33.695" y="33.385" smashed="yes" rot="R270">
+<element name="C10" library="rc-master-smd" package="C0603" value="1µF" x="33.695" y="33.385" smashed="yes" rot="R270">
 <attribute name="NAME" x="33.336" y="31.784" size="0.8128" layer="25" ratio="18" rot="R270"/>
 <attribute name="VALUE" x="32.171" y="34.909" size="0.6096" layer="27" ratio="10" rot="R270"/>
@@
 <attribute name="VALUE" x="54.524" y="25.476" size="0.6096" layer="27" ratio="10" rot="R90"/>
 </element>
-<element name="C6" library="rc-master-smd" package="C1206" value="1µF,50V" x="50.9" y="21.9" rot="R180"/>
+<element name="C6" library="rc-master-smd" package="C1206" value="10µF,50V" x="50.9" y="21.9" rot="R180"/>
 <element name="VMOT" library="SparkFun" package="1X02_NO_SILK" value="" x="1.89" y="18.14" smashed="yes">
 <attribute name="NAME" x="0.9438" y="19.3688" size="1.016" layer="25"/>
